Commit message: Base model

File: summit_description/robot/summit.urdf.xacro (robot description, xacro)
@@ -10,16 +10,17 @@
 	<xacro:macro name="robot">
 		<xacro:summit_base/>
-		<xacro:omni_wheel prefix="summit_front_right" parent="summit_base_footprint" reflect="false">
+		<xacro:omni_wheel prefix="summit_front_right" parent="summit_base_link" reflect="false">
 			<origin xyz="${wheel_offset_x} -${wheel_offset_y} ${wheel_offset_z}" rpy="0 0 0"/>
 		</xacro:omni_wheel>
-		<xacro:omni_wheel prefix="summit_front_left" parent="summit_base_footprint" reflect="true">
+		<xacro:omni_wheel prefix="summit_front_left" parent="summit_base_link" reflect="true">
 			<origin xyz="${wheel_offset_x} ${wheel_offset_y} ${wheel_offset_z}" rpy="0 0 0"/>
 		</xacro:omni_wheel>
-		<xacro:omni_wheel prefix="summit_back_left" parent="summit_base_footprint" reflect="true">
+		<xacro:omni_wheel prefix="summit_back_left" parent="summit_base_link" reflect="true">
 			<origin xyz="-${wheel_offset_x} ${wheel_offset_y} ${wheel_offset_z}" rpy="0 0 0"/>
 		</xacro:omni_wheel>
-		<xacro:omni_wheel prefix="summit_back_right" parent="summit_base_footprint" reflect="false">
+		<xacro:omni_wheel prefix="summit_back_right" parent="summit_base_link" reflect="false">
 			<origin xyz="-${wheel_offset_x} -${wheel_offset_y} ${wheel_offset_z}" rpy="0 0 0"/>
 		</xacro:omni_wheel>
+        <xacro:omni_steering/>
    </xacro:macro>
    <xacro:robot/>

File: summit_description/urdf/base/summit_base.urdf.xacro (robot description, xacro)
@@ -2,21 +2,45 @@
 <robot name="summit_xl" xmlns:xacro="http://www.ros.org/wiki/xacro">
   <xacro:macro name="summit_base">
-	  <!-- Robot mechanical and motor parameters -->
-	  <xacro:property name="PI" value="3.1415926535897931"/>
-	  <xacro:property name="wheel_width" value="0.175" />
-	<!-- BASE FOOTPRINT -->
-		<link name="summit_base_footprint">
-		  <visual>
-			  <origin xyz="0 0 0" rpy="0 0 0" />
-			  <geometry>
-				 <box size="0.001 0.001 0.001" />
-			  </geometry>
-		  </visual>
-          <inertial>
-            <mass value="125.0" />
-            <origin xyz="0 0 0" />
-            <inertia  ixx="1.391" ixy="0.004"  ixz="0.0"  iyy="6.853"  iyz="0.0"  izz="6.125" />
-        </inertial>
-		</link>
+    <xacro:include filename="$(find summit_description)/urdf/base/summit_base.gazebo.xacro" />
+    <!-- Robot mechanical and motor parameters -->
+    <xacro:property name="PI" value="3.1415926535897931"/>
+    <xacro:property name="wheel_width" value="0.175" />
+    <!-- BASE FOOTPRINT -->
+    <link name="summit_base_footprint">
+        <visual>
+            <origin xyz="0 0 0" rpy="0 0 0" />
+            <geometry>
+                <box size="0.001 0.001 0.001" />
+            </geometry>
+        </visual>
+    </link>
+    <joint name="summit_base_footprint_joint" type="fixed">
+        <origin xyz="0 0 ${wheel_radius}" rpy="0 0 0" /> <!-- ${wheel_radius} property must be defined inside wheel description -->
+        <parent link="summit_base_footprint"/>
+        <child link="summit_base_link" />
+    </joint>
+  <!-- BASE_LINK -->
+  <link name="summit_base_link">
+    <inertial>
+      <mass value="125.0" />
+      <origin xyz="0 0 0" />
+      <inertia  ixx="1.391" ixy="0.004"  ixz="0.0"  iyy="6.853"  iyz="0.0"  izz="6.125" />
+    </inertial>
+    <visual>
+       <origin xyz="0 0 0" rpy="0 0 0" />
+       <geometry>
+	     <mesh filename="package://summit_description/meshes/base/summit_base.dae"/>
+       </geometry>
+       <material name="darkgrey">
+         <color rgba="0.1 0.1 0.1 1"/>
+       </material>
+    </visual>
+    <collision>
+       <origin xyz="0 0 0" rpy="0 0 0 " />
+       <geometry>
+         <mesh filename="package://summit_description/meshes/base/summit_base.dae"/>
+       </geometry>
+    </collision>
+  </link>
   </xacro:macro>
 </robot>
